File: PCB/SensorPresion/SensorPresion.sch (KiCad schematic (older format))
At the start: 60 parts, among them J1 USB_B_Micro, J2 Conn_01x05_Female, SW1 SW_DPST_x2, U1 OPAMP, U10 OPAMP, U11 TP4056, U12 DW01, U13 FS8205A, U14 PIC16F882-IP, U15 BLUETOOTH-SERIAL-HC-06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

Commit message: PCB Footprints
Parts:
- J1: symbol Connector:USB_B_Micro -> SensorPresion-rescue:USB_B_Micro-Connector
- U11: symbol TP4056:TP4056 -> SensorPresion-rescue:TP4056-TP4056
- U12: symbol DW01:DW01 -> SensorPresion-rescue:DW01-DW01
- U13: symbol FS8205A:FS8205A -> SensorPresion-rescue:FS8205A-FS8205A
- U15: symbol HC-06:BLUETOOTH-SERIAL-HC-06 -> SensorPresion-rescue:BLUETOOTH-SERIAL-HC-06-HC-06
- gave numbers to parts that had none: 1
Changed lines of the file:
@@
 s_signal_8
 $Comp
-L TP4056:TP4056 U11
+L SensorPresion-rescue:TP4056-TP4056 U11
 U 1 1 614B27FE
 P 3550 4400
@@
 $EndComp
 $Comp
-L DW01:DW01 U12
+L SensorPresion-rescue:DW01-DW01 U12
 U 1 1 614B3019
 P 5350 4300
@@
 $EndComp
 $Comp
-L FS8205A:FS8205A U13
+L SensorPresion-rescue:FS8205A-FS8205A U13
 U 1 1 614B3B9A
 P 5350 5600
@@
 	6250 4400 6400 4400
 $Comp
-L Connector:USB_B_Micro J1
+L SensorPresion-rescue:USB_B_Micro-Connector J1
 U 1 1 615686B9
 P 1250 4500
@@
 Connection ~ 5450 6200
 $Comp
-L HC-06:BLUETOOTH-SERIAL-HC-06 U15
+L SensorPresion-rescue:BLUETOOTH-SERIAL-HC-06-HC-06 U15
 U 1 1 61736AFF
 P 12150 2100
@@
 $EndComp
 $Comp
-L Connector:Conn_01x02_Female J?
+L Connector:Conn_01x02_Female J3
 U 1 1 6144C19B
 P 1350 2700
-F 0 "J?" H 1378 2676 50  0000 L CNN
+F 0 "J3" H 1378 2676 50  0000 L CNN
 F 1 "Conn_01x02_Female" H 1378 2585 50  0000 L CNN
 F 2 "" H 1350 2700 50  0001 C CNN
